Commit message: camera added

File: resource/LD90.urdf (robot description, URDF)
Before this commit: robot LD90, 0 links, 0 joints
Links:
- added link oakd_rgb_camera_link, mass 0.010; collision box size=0.05 0.05 0.05; visual box size=0.05 0.05 0.05
Joints:
- added joint oakd_rgb_camera_joint: type fixed, parent base_link, child oakd_rgb_camera_link, origin xyz=0.058400 0.000000 0.096760 rpy=-0.577350 0.577350 -0.577350

Commit message: transfered from map branchD

File: resource/LD90.urdf (robot description, URDF)
Before this commit: robot LD90, 1 links, 1 joints
Links:
- removed link oakd_rgb_camera_link
Joints:
- removed joint oakd_rgb_camera_joint
